Commit message: 运动学控制整体框架搭建完成

File: assets/bookarm_urdf/urdf/bookarm_urdf.urdf (robot description, URDF)
Before this commit: robot bookarm_urdf, 7 links, 6 joints
Joints:
- joint joint1_base: limit lower=0 upper=0 effort=0 velocity=0 -> lower=-3.14159 upper=3.14159 effort=1 velocity=1
- joint joint2_shoulder: limit lower=0 upper=0 effort=0 velocity=0 -> lower=-1.5708 upper=1.5708 effort=1 velocity=1
- joint joint3_elbow: limit lower=0 upper=0 effort=0 velocity=0 -> lower=-3.14159 upper=1.5708 effort=1 velocity=1
- joint joint4_wrist: limit lower=0 upper=0 effort=0 velocity=0 -> lower=-1.8 upper=2.35619 effort=1 velocity=1
- joint joint_pole: limit lower=0 upper=0 effort=0 velocity=0 -> lower=-2.0944 upper=2.0944 effort=1 velocity=1

Commit message: 正逆运动学测试正确，完成逆解抓取效果

File: assets/bookarm_urdf/urdf/bookarm_urdf.urdf (robot description, URDF)
Before this commit: robot bookarm_urdf, 7 links, 6 joints
Joints:
- joint joint2_shoulder: limit lower=-1.5708 upper=1.5708 effort=1 velocity=1 -> lower=-1.59 upper=1.69 effort=1 velocity=1
- joint joint3_elbow: limit lower=-3.14159 upper=1.5708 effort=1 velocity=1 -> lower=-2.78 upper=1.7 effort=1 velocity=1
- joint joint4_wrist: limit lower=-1.8 upper=2.35619 effort=1 velocity=1 -> lower=-2.04 upper=2.1 effort=1 velocity=1
- joint joint_pole: limit lower=-2.0944 upper=2.0944 effort=1 velocity=1 -> lower=-1.26 upper=1.94 effort=1 velocity=1
